File: pcb-business-card.kicad_pcb (KiCad board)
At the start: 2 copper layers, 54 x 85.6 mm, 715 parts

Commit message: Added notes and a preview
Other:
- board text added: "Your awesone brand / catchphrase / artwork! Cyril Lugan (CC-BY)"
Changed lines of the file:
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@@
   (general
     (thickness 1.6)
-    (drawings 87)
+    (drawings 88)
     (tracks 0)
     (zones 0)
@@
     (visible_elements FFFFFF7F)
     (pcbplotparams
-      (layerselection 0x010fc_ffffffff)
+      (layerselection 0x010f0_ffffffff)
       (usegerberextensions false)
       (usegerberattributes false)
@@
       (drillshape 0)
       (scaleselection 1)
-      (outputdirectory "Gerber v1/"))
+      (outputdirectory "gerbers/"))
   )
   (net 0 "")
@@
       (effects (font (size 1 1) (thickness 0.15)))
     )
-    (fp_circle (center 0 0) (end 2.25 0) (layer Cmts.User) (width 0.15))
     (fp_circle (center 0 0) (end 2.5 0) (layer F.CrtYd) (width 0.05))
+    (fp_circle (center 0 0) (end 2.25 0) (layer Cmts.User) (width 0.15))
     (fp_text user %R (at 0.3 0) (layer F.Fab) hide
       (effects (font (size 1 1) (thickness 0.15)))
@@
     (pad 1 smd rect (at 0 0) (size 1.08 1.08) (layers F.Cu F.Paste F.Mask))
   )
+  (gr_text "Your awesone\nbrand / catchphrase / artwork!\n\nCyril Lugan (CC-BY)" (at 127.254 65.024) (layer F.SilkS)
+    (effects (font (size 1.5 1.5) (thickness 0.3)) (justify left))
+  )
   (gr_poly (pts (xy 144.78 136.525) (xy 177.165 136.525) (xy 177.165 143.51) (xy 144.78 143.51)) (layer F.SilkS) (width 0.15))
